File: IrDA_RS232.kicad_pcb (KiCad board)
At the start: 4 copper layers, 62.9 x 32 mm, 36 parts, among them J1 RS232, U1 MAX232, U2 MAX232, U3 MCP2155, U4 TFDU4301, Y1 11.0592 MHz

Commit message: add gerbers and PDF
Parts:
- added D2: BAV99, Package_TO_SOT_SMD:SOT-23, F.Cu at (46.9, 49.5)
- added Q1: 2N7002, Package_TO_SOT_SMD:SOT-23, F.Cu at (51.9, 49.5)
- added R7: 10k, Resistor_SMD:R_0402_1005Metric, F.Cu at (45.5, 51.8)
- added R8: 100k, Resistor_SMD:R_0402_1005Metric, F.Cu at (49.4, 48.8)
- added R9: 10k, Resistor_SMD:R_0402_1005Metric, F.Cu at (65.9, 50.5)
Connections:
- U3 pad 9: +5V -> /MCP_RI
Routing:
- net /RS232_RING: track 0.00 -> 34.5 mm, vias 0 -> 1
- net /MCP_RI: track 0.00 -> 14.0 mm
- net /MCP_TX: track 29.8 -> 39.3 mm, vias 0 -> 2
- net Net-(D2-Pad3): track 0.00 -> 8.71 mm
- net GND: track 33.8 -> 41.4 mm, vias 27 -> 36
- net /MCP_RX: track 30.5 -> 27.4 mm, vias 0 -> 2
- net +5V: track 41.2 -> 40.5 mm, vias 24 -> 26
Other:
- board text added: "tbspace.de"
